File: CAN-Board-V1/CAN-Board-V1.kicad_pcb (KiCad board)
At the start: 2 copper layers, 63.5 x 50.8 mm, 8 parts, among them U1 MCP2551-I-P, U2 MCP2515-I_P, Y1 8Mhz

Commit message: V1 Complete
Parts:
- added C3: CP_Small, Capacitor_THT:C_Disc_D5.0mm_W2.5mm_P2.50mm, F.Cu at (129.0, 52.8)
- added C4: 0.1uF, Capacitor_THT:C_Disc_D5.0mm_W2.5mm_P2.50mm, F.Cu at (133.1, 52.8)
- added C5: .1uF, Capacitor_THT:C_Disc_D5.0mm_W2.5mm_P2.50mm, F.Cu at (125.0, 52.8)
- added D1: LED_Small, LED_THT:LED_D5.0mm, F.Cu at (125.2, 45.5)
- added G***: LOGO, SolderMasks:Face, F.Cu at (93.4, 62.0)
- added G***: LOGO, SolderMasks:GhostSmall, F.Cu at (124.3, 75.1)
- added H1: MountingHole, MountingHole:MountingHole_3.2mm_M3, F.Cu at (133.1, 44.7)
- added H2: MountingHole, MountingHole:MountingHole_3.2mm_M3, F.Cu at (133.1, 82.3)
- added H3: MountingHole, MountingHole:MountingHole_3.2mm_M3, F.Cu at (82.8, 44.7)
- added H4: MountingHole, MountingHole:MountingHole_3.2mm_M3, F.Cu at (82.8, 82.3)
- added J1: Conn_01x07_Male, Connector_PinHeader_1.27mm:PinHeader_1x07_P1.27mm_Vertical, F.Cu at (137.8, 66.0)
- added J2: Screw_Terminal_01x02, TerminalBlock_TE-Connectivity:TerminalBlock_TE_282834-2_1x02_P2.54mm_Horizontal, F.Cu at (101.1, 41.7)
- added J3: Screw_Terminal_01x02, TerminalBlock_TE-Connectivity:TerminalBlock_TE_282834-2_1x02_P2.54mm_Horizontal, F.Cu at (108.3, 41.7)
- added J4: Screw_Terminal_01x02, TerminalBlock_TE-Connectivity:TerminalBlock_TE_282834-2_1x02_P2.54mm_Horizontal, F.Cu at (115.6, 41.7)
- added R3: 500k, Resistor_THT:R_Axial_DIN0207_L6.3mm_D2.5mm_P10.16mm_Horizontal, F.Cu at (116.8, 49.3)
- added R4: 120, Resistor_THT:R_Axial_DIN0207_L6.3mm_D2.5mm_P10.16mm_Horizontal, F.Cu at (87.6, 41.1)
- C1, C2: value C_Small -> 22uF; footprint Capacitor_SMD:C_01005_0402Metric -> Capacitor_THT:C_Disc_D5.0mm_W2.5mm_P2.50mm
- R1, R2: footprint Resistor_SMD:R_0603_1608Metric -> Resistor_THT:R_Axial_DIN0207_L6.3mm_D2.5mm_P10.16mm_Horizontal
- U1: footprint Package_DIP:DIP-8_W7.62mm -> Package_DIP:DIP-8_W7.62mm_Socket
- U2: footprint Package_DIP:DIP-18_W7.62mm -> Package_DIP:DIP-18_W7.62mm_Socket
- moved R1 22.7 mm to (106.7, 55.2), turned to 0 degrees
- moved C1 19.8 mm to (94.0, 68.8), turned to -90 degrees
- moved C2 18.1 mm to (94.0, 78.1), turned to 90 degrees
- moved Y1 17.9 mm to (88.3, 76.2)
- moved R2 15.0 mm to (85.3, 49.3)
- moved U1 14.0 mm to (89.5, 53.3)
- moved U2 14.0 mm to (101.6, 60.3)
- moved G*** 1.12 mm to (107.5, 63.9)
Connections:
- net +5V renamed VCC
- U1 pad 5: Net-(U1-Pad5) -> unconnected-(U1-Vref-Pad5)
- U2 pad 10: Net-(U2-Pad10) -> unconnected-(U2-*RX1BF-Pad10)
- U2 pad 11: Net-(U2-Pad11) -> unconnected-(U2-*RX0BF-Pad11)
- U2 pad 3: Net-(U2-Pad3) -> unconnected-(U2-CLKOUT/SOF-Pad3)
- U2 pad 4: Net-(U2-Pad4) -> unconnected-(U2-*TX0RTS-Pad4)
- U2 pad 5: Net-(U2-Pad5) -> unconnected-(U2-*TX1RTS-Pad5)
- U2 pad 6: Net-(U2-Pad6) -> unconnected-(U2-*TX2RTS-Pad6)
Routing:
- net Earth: track 43.3 -> 125.9 mm, vias 2 -> 0
- net VCC: track 24.9 -> 74.2 mm
- net CANH: track 0.00 -> 33.8 mm
- net Net-(J1-Pin_1): track 0.00 -> 32.5 mm
- net Net-(J1-Pin_2): track 0.00 -> 32.0 mm
- net Net-(J1-Pin_3): track 0.00 -> 31.5 mm
- net Net-(J1-Pin_4): track 0.00 -> 30.9 mm
- net Net-(J1-Pin_5): track 0.00 -> 30.4 mm
- net CANL: track 0.00 -> 30.0 mm
- net Net-(D1-A): track 0.00 -> 7.67 mm
- net Net-(U2-*RESET): track 5.26 -> 11.9 mm
- net Net-(U2-OSC2): track 10.9 -> 15.1 mm
- net Net-(J2-Pin_1): track 0.00 -> 3.76 mm
- net Net-(U2-OSC1): track 12.2 -> 14.6 mm
- net Net-(U1-RXD): track 11.4 -> 13.7 mm
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Other:
- net class Default removed
- board text added: "*CS"
- board text added: "*INT"
- board text added: "->"
- board text added: "CAN Board Rev 1 10/20/23"
- board text added: "Developed By: Andrew McGhee https://github.com/AndrewMcGhee"
- board text added: "GND"
- board text added: "SCK"
- board text added: "SI"
- board text added: "SO"
- board text added: "To Microcontroller"
- board text added: "Vcc"

Commit message: mian
Parts:
- C3: value CP_Small -> 10uF
- J1: footprint Connector_PinHeader_1.27mm:PinHeader_1x07_P1.27mm_Vertical -> Connector_PinHeader_2.00mm:PinHeader_1x07_P2.00mm_Vertical
- R3: value 500k -> 500
- moved J1 2.54 mm to (137.8, 68.6)
Routing:
- net VCC: track 74.2 -> 75.0 mm
- net Net-(J1-Pin_1): track 32.5 -> 33.2 mm
- net Net-(J1-Pin_2): track 32.0 -> 32.5 mm
