File: CAN-Board-V1/CAN-Board-V1.kicad_sch (KiCad schematic)
At the start: 21 parts, among them J1 Conn_01x07_Male, J2 Screw_Terminal_01x02, J3 Screw_Terminal_01x02, J4 Screw_Terminal_01x02, U1 MCP2551-I-P, U2 MCP2515-I_P, Y1 8Mhz

Commit message: Updated
Parts:
- R3: value 500k -> 500
Changed lines of the file:
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@@
       (effects (font (size 1.27 1.27)))
     )
-    (property "Value" "500k" (at 41.91 83.693 90)
+    (property "Value" "500" (at 41.91 83.693 90)
       (effects (font (size 1.27 1.27)))
     )

Commit message: mian
Parts:
- J1: footprint Connector_PinHeader_1.27mm:PinHeader_1x07_P1.27mm_Vertical -> Connector_PinHeader_2.00mm:PinHeader_1x07_P2.00mm_Vertical
Changed lines of the file:
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@@
       (effects (font (size 1.27 1.27)) (justify right))
     )
-    (property "Footprint" "Connector_PinHeader_1.27mm:PinHeader_1x07_P1.27mm_Vertical" (at 172.72 49.53 0)
+    (property "Footprint" "Connector_PinHeader_2.00mm:PinHeader_1x07_P2.00mm_Vertical" (at 172.72 49.53 0)
       (effects (font (size 1.27 1.27)) hide)
     )
